File: STM32F4 Test Board/STM32F4 Test Board.kicad_sch (KiCad schematic)
At the start: 20 parts, among them U1 STM32F405RGTx

Commit message: The schematic part of the board is completed.
Parts:
- added C13, C14, C16: 12p, symbol Device:C_Polarized_US
- added C15: 12u, symbol Device:C_Polarized_US
- added D3: DIODE, Diode_THT:D_DO-35_SOD27_P7.62mm_Horizontal, symbol Diode:BAV20
- added D4: LED, symbol Device:LED
- added FB1: 600@600MHz, symbol Device:FerriteBead
- added H1, H2, H3, H4: MountingHole_Pad, symbol Mechanical:MountingHole_Pad
- added J1: USB_B_Micro, symbol Connector:USB_B_Micro
- added J2: Screw_Terminal_01x02, symbol Connector:Screw_Terminal_01x02
- added J3: Conn_01x10, symbol Connector_Generic:Conn_01x10
- added J4, J5: Screw_Terminal_01x04, symbol Connector:Screw_Terminal_01x04
- added Q1: AO3401A, digikey-footprints:SOT-23-3, symbol dk_Transistors-FETs-MOSFETs-Single:AO3401A
- added R4: 47, symbol Device:R
- added R5: 10K, symbol Device:R
- added R6: 47K, symbol Device:R
- added R7: 15K, symbol Device:R
- added R8: 270, symbol Device:R
- added R9: 1K, symbol Device:R
- added SW1: SW_SPDT, symbol Switch:SW_SPDT
- added TH1: 250mA, symbol Device:Thermistor
- added U2: AP65111AWU, Package_TO_SOT_SMD:TSOT-23-6, symbol Regulator_Switching:AP65111AWU
- added U3: USBLC6-2SC6, Package_TO_SOT_SMD:SOT-23-6, symbol Power_Protection:USBLC6-2SC6
- added Y1: 16MHz, symbol Device:Crystal_GND23
Connections:
- net +3.3V: now also D4.2 (A), J3.1 (Pin_1), J4.1 (Pin_1), J5.1 (Pin_1), R6.2, SW1.1 (A)
- net BOOT0: now also R5.2
- net BUCK_EN: now also U2.5 (EN)
- net BUCK_IN: now also C15.1, FB1.2, U2.1 (IN)
- net BUCK_SW: now also C16.1, U2.3 (SW)
- net GND: now also C13.2, C14.2, C15.2, H1.1, H2.1, H3.1, H4.1, J1.5 (GND), J2.2 (Pin_2), J3.3 (Pin_3), J3.5 (Pin_5), J3.9 (Pin_9), J4.4 (Pin_4), J5.4 (Pin_4), Q1.1 (G), R8.1, R9.1, SW1.3 (C), U2.2 (GND), U3.2 (GND), Y1.2, Y1.3
- net HSE_IN: now also R4.2
- net HSE_OUT: now also C13.1, Y1.1
- net I2C1_SCL: now also J4.2 (Pin_2)
- net I2C1_SDA: now also J4.3 (Pin_3)
- net NRST: now also J3.10 (Pin_10)
- net SWCLK: now also J3.4 (Pin_4)
- net USART3_RX: now also J5.3 (Pin_3)
- net USART3_TX: now also J5.2 (Pin_2)
- net USB_D+: now also U3.4 (I/O2)
- net USB_D-: now also U3.6 (I/O1)
- new net: R7.1, R8.2
- new net: D3.1 (K), FB1.1, Q1.2 (S)
- new net: Q1.3 (D), TH1.2
- new net: R5.1, SW1.2 (B)
- new net: C14.1, R4.1, Y1.4
- new net: D4.1 (K), R9.2
- new net +12V: J2.1 (Pin_1), TH1.1
- new net +5V: D3.2 (A), J1.1 (VBUS), U3.5 (VBUS)
- new net BUCJK_BST: C16.2
- new net BUCK_FB: R6.1, R7.2, U2.6 (FB)
- new net BUCK_SWT: U2.4 (BST)
- new net SW0: J3.6 (Pin_6)
- new net SWDI0: J3.2 (Pin_2)
- new net USB_CONN_D+: J1.3 (D+), U3.3 (I/O2)
- new net USB_CONN_D-: J1.2 (D-), U3.1 (I/O1)
- no-connect marks 40 -> 44
Other:
- note added: "BIRIMLER"
- note added: "CONNECTORS"
- note added: "OSILATOR DEVRESI"
- note added: "POWER SYSTEM"
- moved on the sheet: C10, C11, C12, C3, C4, C5, C6, C7, C8, C9, D1, D2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
